File: loraNode.brd (EAGLE design)
At the start: 33.2 x 23.4 mm, 3 parts

Commit message: Update board.2
Routing:
- net GND: track 20.1 -> 14.1 mm
Changed lines of the file:
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@@
 <wire x1="5.77" y1="2.17" x2="2.89" y2="2.17" width="0.8128" layer="1"/>
 <wire x1="7.11" y1="3.51" x2="5.77" y2="2.17" width="0.8128" layer="1"/>
-<wire x1="24.16" y1="5.51" x2="29.25" y2="5.51" width="0.8128" layer="1"/>
-<wire x1="29.25" y1="5.51" x2="29.9" y2="4.86" width="0.8128" layer="1"/>
 <polygon width="0.8128" layer="1">
-<vertex x="0.25" y="0.1"/>
-<vertex x="0.25" y="23"/>
-<vertex x="0.35" y="23.1"/>
-<vertex x="33.3" y="23.1"/>
-<vertex x="33.35" y="23.05"/>
-<vertex x="33.35" y="0.15"/>
-<vertex x="0.3" y="0.15"/>
+<vertex x="-0.1" y="0.05"/>
+<vertex x="-0.1" y="23.05"/>
+<vertex x="0.15" y="23.3"/>
+<vertex x="33.1" y="23.3"/>
+<vertex x="33.1" y="0.05"/>
 </polygon>
 </signal>
